File: ch32v003j4m6-breakout.kicad_sch (KiCad schematic)
At the start: 3 parts, among them J1 Conn_01x04, J2 Conn_01x04, U1 CH32V003J4M6

Commit message: fix: exclude headers from BOM
Parts:
- J1, J2: now left out of the parts list
Changed lines of the file:
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@@
 		(unit 1)
 		(exclude_from_sim no)
-		(in_bom yes)
+		(in_bom no)
 		(on_board yes)
 		(dnp no)
@@
 		(unit 1)
 		(exclude_from_sim no)
-		(in_bom yes)
+		(in_bom no)
 		(on_board yes)
 		(dnp no)
